Commit message: added modified urdf & xacro files

File: my_robot_description/urdf/arm.xacro (robot description, xacro)
@@ -9,69 +9,69 @@
     <xacro:property name="hand_length" value="0.3" />
     <link name="arm_base_link">
-           <visual>
-               <geometry>
-                   <box size="${arm_base_length} ${arm_base_width} ${arm_base_height}"/>
-               </geometry>
-               <origin xyz="0 0 ${arm_base_height / 2.0}" rpy="0 0 0"/>
-               <material name="orange" />
-             </visual>
-            <collision>
-               <geometry>
-                   <box size="${arm_base_length} ${arm_base_width} ${arm_base_height}"/>
-               </geometry>
-               <origin xyz="0 0 ${arm_base_height / 2.0}" rpy="0 0 0"/>
-            </collision>
-            <xacro:box_inertia m="0.5" x="${arm_base_length}" y="${arm_base_width}" z="${arm_base_height}"
-                               o_xyz="0 0 ${arm_base_height / 2.0}" o_rpy="0 0 0" />
+        <visual>
+            <geometry>
+                <box size="${arm_base_length} ${arm_base_width} ${arm_base_height}" />
+            </geometry>
+            <origin xyz="0 0 ${arm_base_height / 2.0}" rpy="0 0 0" />
+            <material name="orange" />
+        </visual>
+        <collision>
+            <geometry>
+                <box size="${arm_base_length} ${arm_base_width} ${arm_base_height}" />
+            </geometry>
+            <origin xyz="0 0 ${arm_base_height / 2.0}" rpy="0 0 0" />
+        </collision>
+        <xacro:box_inertia m="0.5" x="${arm_base_length}" y="${arm_base_width}" z="${arm_base_height}"
+                           o_xyz="0 0 ${arm_base_height / 2.0}" o_rpy="0 0 0" />
     </link>
     <link name="forearm_link">
-           <visual>
-               <geometry>
-                   <cylinder radius="${forearm_radius}" length= "${forearm_length}" />
-               </geometry>
-               <origin xyz="0 0 ${forearm_length / 2.0}" rpy="0 0 0"/>
-               <material name="yellow" />
-           </visual>
-           <collision>
-                <geometry>
-                   <cylinder radius="${forearm_radius}" length= "${forearm_length}" />
-               </geometry>
-               <origin xyz="0 0 ${forearm_length / 2.0}" rpy="0 0 0"/>
-           </collision>
-           <xacro:cylinder_inertia m="0.3" r="${forearm_radius}" l="${forearm_length}"
-                                   o_xyz="0 0 ${forearm_length / 2.0}" o_rpy="0 0 0" />
+        <visual>
+            <geometry>
+                <cylinder radius="${forearm_radius}" length="${forearm_length}" />
+            </geometry>
+            <origin xyz="0 0 ${forearm_length / 2.0}" rpy="0 0 0" />
+            <material name="yellow" />
+        </visual>
+        <collision>
+            <geometry>
+                <cylinder radius="${forearm_radius}" length="${forearm_length}" />
+            </geometry>
+            <origin xyz="0 0 ${forearm_length / 2.0}" rpy="0 0 0" />
+        </collision>
+        <xacro:cylinder_inertia m="0.3" r="${forearm_radius}" l="${forearm_length}"
+                                o_xyz="0 0 ${forearm_length / 2.0}" o_rpy="0 0 0" />
     </link>
     <link name="hand_link">
-           <visual>
-               <geometry>
-                   <cylinder radius="${hand_radius}" length= "${hand_length}" />
-               </geometry>
-               <origin xyz="0 0 ${hand_length / 2.0}" rpy="0 0 0"/>
-               <material name="orange" />
-           </visual>
-           <collision>
-                <geometry>
-                   <cylinder radius="${hand_radius}" length= "${hand_length}" />
-               </geometry>
-               <origin xyz="0 0 ${hand_length / 2.0}" rpy="0 0 0"/>
-           </collision>
-           <xacro:cylinder_inertia m="0.3" r="${hand_radius}" l="${hand_length}"
-                                   o_xyz="0 0 ${hand_length / 2.0}" o_rpy="0 0 0" />
+        <visual>
+            <geometry>
+                <cylinder radius="${hand_radius}" length="${hand_length}" />
+            </geometry>
+            <origin xyz="0 0 ${hand_length / 2.0}" rpy="0 0 0" />
+            <material name="orange" />
+        </visual>
+        <collision>
+            <geometry>
+                <cylinder radius="${hand_radius}" length="${hand_length}" />
+            </geometry>
+            <origin xyz="0 0 ${hand_length / 2.0}" rpy="0 0 0" />
+        </collision>
+        <xacro:cylinder_inertia m="0.3" r="${hand_radius}" l="${hand_length}"
+                                o_xyz="0 0 ${hand_length / 2.0}" o_rpy="0 0 0" />
     </link>
     <joint name="arm_base_forearm_joint" type="revolute">
-           <parent link="arm_base_link"/>
-           <child link="forearm_link"/>
-           <origin xyz="0 0 ${arm_base_height}" rpy="0 0 0"/>
-           <axis xyz="0 1 0"/>
-           <limit lower="0" upper="${pi/2}" effort="100" velocity="100"/>
-           <dynamics friction="0.3" damping="0.3" />
+        <parent link="arm_base_link" />
+        <child link="forearm_link" />
+        <origin xyz="0 0 ${arm_base_height}" rpy="0 0 0" />
+        <axis xyz="0 1 0" />
+        <limit lower="0" upper="${pi/2}" effort="100" velocity="100" />
+        <dynamics friction="0.3" damping="0.3" />
     </joint>
     <joint name="forearm_hand_joint" type="revolute">
-           <parent link="forearm_link"/>
-           <child link="hand_link"/>
-           <origin xyz="0 0 ${forearm_length}" rpy="0 0 0"/>
-           <axis xyz="0 1 0"/>
-           <limit lower="0" upper="${pi/2}" effort="100" velocity="100"/>
-           <dynamics friction="0.3" damping="0.3" />
+        <parent link="forearm_link" />
+        <child link="hand_link" />
+        <origin xyz="0 0 ${forearm_length}" rpy="0 0 0" />
+        <axis xyz="0 1 0" />
+        <limit lower="0" upper="${pi/2}" effort="100" velocity="100" />
+        <dynamics friction="0.3" damping="0.3" />
     </joint>
 </robot>

File: my_robot_description/urdf/camera.xacro (robot description, xacro)
@@ -6,12 +6,12 @@
     <link name="camera_link">
         <visual>
-           <geometry>
-                <box size="${camera_length} ${camera_width} ${camera_height}"/>
-           </geometry>
-           <material name="grey" />
+            <geometry>
+                <box size="${camera_length} ${camera_width} ${camera_height}" />
+            </geometry>
+            <material name="grey" />
         </visual>
         <collision>
             <geometry>
-                <box size="${camera_length} ${camera_width} ${camera_height}"/>
+                <box size="${camera_length} ${camera_width} ${camera_height}" />
             </geometry>
         </collision>
@@ -20,40 +20,34 @@
     </link>
     <joint name="base_camera_joint" type="fixed">
-         <parent link="base_link"/>
-         <child link="camera_link"/>
-         <origin xyz="${(base_length + camera_length)/2} 0 ${base_height/2}" rpy="0 0 0" />
+        <parent link="base_link" />
+        <child link="camera_link" />
+        <origin xyz="${(base_length + camera_length) / 2.0} 0 ${base_height / 2.0}" rpy="0 0 0" />
     </joint>
-    <link name="camera_link_optical"/>
+    <link name="camera_link_optical" />
     <joint name="camera_optical_joint" type="fixed">
-         <origin xyz="0 0 0" rpy="${-pi/2} 0 ${-pi/2}"/>
-         <parent link="camera_link"/>
-         <child link="camera_link_optical"/>
+        <origin xyz="0 0 0" rpy="${-pi/2} 0 ${-pi/2}"/>
+        <parent link="camera_link"/>
+        <child link="camera_link_optical"/>
     </joint>
     <gazebo reference="camera_link">
-        <sensor name="camera" type="camera">
-            <camera>
-                <horizontal_fov>1.3962634</horizontal_fov>
-                <image>
-                    <width>640</width>
-                    <height>480</height>
-                    <format>R8G8B8</format>
-                </image>
-                <clip>
-                    <near>0.1</near>
-                    <far>15</far>
-                </clip>
-                <noise>
-                    <type>gaussian</type>
-                    <mean>0.0</mean>
-                    <stddev>0.007</stddev>
-                </noise>
-                <optical_frame_id>camera_link_optical</optical_frame_id>
-                <camera_info_topic>camera/camera_info</camera_info_topic>
-            </camera>
-            <always_on>1</always_on>
-            <update_rate>20</update_rate>
-            <visualize>true</visualize>
-            <topic>camera/image_raw</topic>
-        </sensor>
+    <sensor name="camera" type="camera">
+        <camera>
+            <horizontal_fov>1.3962634</horizontal_fov>
+            <image>
+                <width>640</width>
+                <height>480</height>
+                <format>R8G8B8</format>
+            </image>
+            <clip>
+                <near>0.1</near>
+                <far>15</far>
+            </clip>
+            <optical_frame_id>camera_link_optical</optical_frame_id>
+        </camera>
+        <always_on>1</always_on>
+        <update_rate>20</update_rate>
+        <visualize>true</visualize>
+        <topic>camera/image_raw</topic>
+    </sensor>
     </gazebo>
 </robot>

File: my_robot_description/urdf/common_properties.xacro (robot description, xacro)
@@ -8,8 +8,8 @@
     </material>
     <material name="orange">
-        <color rgba="1.0 0.5 0 1"/>
+        <color rgba="1.0 0.5 0 1" />
     </material>
     <material name="yellow">
-        <color rgba="1.0 1.0 0 1"/>
+        <color rgba="1.0 1.0 0 1" />
     </material>
     <xacro:macro name="box_inertia" params="m x y z o_xyz o_rpy">

File: my_robot_description/urdf/my_robot.urdf.xacro (robot description, xacro)
@@ -8,7 +8,7 @@
     <xacro:include filename="camera.xacro" />
     <joint name="mobile_base_arm_joint" type="fixed">
-        <parent link="base_link"/>
-        <child link="arm_base_link"/>
-        <origin xyz="${base_length/4} 0 ${base_height}" rpy="0 0 0"/>
+        <parent link="base_link" />
+        <child link="arm_base_link" />
+        <origin xyz="${base_length / 4.0} 0 ${base_height}" rpy="0 0 0" />
     </joint>
 </robot>

File: my_robot_description/urdf/standalone_arm.urdf.xacro (robot description, xacro)
@@ -3,4 +3,4 @@
     <xacro:include filename="common_properties.xacro" />
     <xacro:include filename="arm.xacro" />
-    <xacro:include filename="arm_gazebo.xacro"/>
+    <xacro:include filename="arm_gazebo.xacro" />
 </robot>
